File: FiveStageMonoEQ.sch (KiCad schematic (older format))
At the start: 72 parts, among them J1 AudioJack3, J2 AudioJack3, U1 LM833, U2 LM833, U3 LM833, U4 LM833, U5 LM833, U6 LM317_T

Commit message: updating PCB design to all SMD and adding multisheet stereo EQ
Parts:
- removed R35: 1800, SamacSys_Parts:RESC2012X60N, symbol FiveStageEQ-rescue:R_Small_US-Device
- removed R37: 240, SamacSys_Parts:RESC1608X55N, symbol FiveStageEQ-rescue:R_Small_US-Device
- removed U6: LM317_T, SamacSys_Parts:TO255P460X1020X2008-3P, symbol FiveStageEQ-rescue:LM317_TO3-Regulator_Linear
- added U6: L7812CV, SamacSys_Parts:TO255P460X1020X2008-3P, symbol dk_PMIC-Voltage-Regulators-Linear:L7805CV
- C1: footprint 100uf_cap:FK20X5R0J107M -> Capacitor_SMD:C_1206_3216Metric_Pad1.42x1.75mm_HandSolder
- C15, C3, C5, C6, C7, C8: footprint SamacSys_Parts:CAPPA1472W54L508D241 -> Capacitor_SMD:C_1206_3216Metric_Pad1.42x1.75mm_HandSolder
- C16: renamed from C17; footprint SamacSys_Parts:CAPPA1472W54L508D241 -> Capacitor_SMD:C_1206_3216Metric_Pad1.42x1.75mm_HandSolder
- C17: renamed from C19; footprint SamacSys_Parts:CAPPA1472W54L508D241 -> Capacitor_SMD:C_1206_3216Metric_Pad1.42x1.75mm_HandSolder
- C18: renamed from C20; footprint SamacSys_Parts:RCE5C1H104J2A2H03B -> SamacSys_Parts:CAPC3216X125N
- C19: renamed from C21; footprint SamacSys_Parts:RCE5C1H104J2A2H03B -> SamacSys_Parts:CAPC3216X125N
- C2: footprint SamacSys_Parts:RCE5C1H104J2A2H03B -> SamacSys_Parts:CAPC3216X125N
- C20: renamed from C22; footprint SamacSys_Parts:RCE5C1H104J2A2H03B -> SamacSys_Parts:CAPC3216X125N
- C21: renamed from C23; footprint SamacSys_Parts:RCE5C1H104J2A2H03B -> SamacSys_Parts:CAPC3216X125N
- C22: renamed from C24; footprint SamacSys_Parts:RCE5C1H104J2A2H03B -> SamacSys_Parts:CAPC3216X125N
- C23: renamed from C25; footprint SamacSys_Parts:CAPPA1472W54L508D241 -> Capacitor_SMD:C_1206_3216Metric_Pad1.42x1.75mm_HandSolder
- C24: renamed from C26; footprint SamacSys_Parts:CAPPA1472W54L508D241 -> Capacitor_SMD:C_1206_3216Metric_Pad1.42x1.75mm_HandSolder
- C25: renamed from C27; value 0.1μ -> 0.33μ; footprint SamacSys_Parts:CAPPA1472W54L508D241 -> Capacitor_SMD:C_0805_2012Metric_Pad1.15x1.40mm_HandSolder
- C26: renamed from C28; footprint SamacSys_Parts:RCE5C1H104J2A2H03B -> SamacSys_Parts:CAPC3216X125N
- C27: renamed from C29; value 1.0μ -> 10μ; footprint SamacSys_Parts:C330C105K5R5TA -> Capacitor_SMD:C_0805_2012Metric_Pad1.15x1.40mm_HandSolder
- R17: footprint footprints:CFR-25JB-52-18K -> SamacSys_Parts:RESC1608X55N
- R24, R25, R26, R27, R36, R8: footprint SamacSys_Parts:RESAD2990W85L1150D460 -> Resistor_SMD:R_0805_2012Metric_Pad1.15x1.40mm_HandSolder
- R28: footprint SamacSys_Parts:RESAD2990W85L1150D460 -> Resistor_SMD:R_0815_2038Metric_Pad1.53x4.00mm_HandSolder
Connections:
- net labels removed: GND-power
- wire segments 233 -> 227
Other:
- note added: "(14-35 Volts)"
- note added: "(tantalum)"
- note removed: "(14-20 Volts)"
- moved on the sheet: C27
