File: FiveStageStereoEQ/Ring_Filter.sch (KiCad schematic (older format))
At the start: 67 parts, among them U301 LM833, U302 LM833, U303 LM833, U304 LM833, U305 LM833, U306 LM833, U307 LM833

Commit message: almost finished, need to fix audio jack footprint
Parts:
- R327: footprint SamacSys_Parts:RK12L12C0A0G -> SamacSys_Parts:3310H001202L
- R328, R330: footprint SamacSys_Parts:P0925NFC15BR1K -> SamacSys_Parts:3310H001202L
- R332: footprint SamacSys_Parts:RK12L12C0C0P -> SamacSys_Parts:3310H001202L
- U301, U302, U303, U304, U305, U306, U307: footprint LM833_Badge:LM833-N-PDIP -> SamacSys_Parts:SOIC127P600X175-8N
Changed lines of the file:
@@
 F 0 "U305" H 6125 4825 50  0000 C CNN
 F 1 "LM833" H 6125 4925 50  0000 C CNN
-F 2 "LM833_Badge:LM833-N-PDIP" H 6025 5075 50  0001 C CNN
+F 2 "SamacSys_Parts:SOIC127P600X175-8N" H 6025 5075 50  0001 C CNN
 F 3 "~" H 6025 5075 50  0001 C CNN
 	1    6025 5075
@@
 F 0 "U301" H 3025 3525 50  0000 C CNN
 F 1 "LM833" H 3025 3625 50  0000 C CNN
-F 2 "LM833_Badge:LM833-N-PDIP" H 2925 3775 50  0001 C CNN
+F 2 "SamacSys_Parts:SOIC127P600X175-8N" H 2925 3775 50  0001 C CNN
 F 3 "~" H 2925 3775 50  0001 C CNN
 	1    2925 3775
@@
 F 0 "U303" H 6125 2425 50  0000 C CNN
 F 1 "LM833" H 6125 2525 50  0000 C CNN
-F 2 "LM833_Badge:LM833-N-PDIP" H 6025 2675 50  0001 C CNN
+F 2 "SamacSys_Parts:SOIC127P600X175-8N" H 6025 2675 50  0001 C CNN
 F 3 "~" H 6025 2675 50  0001 C CNN
 	1    6025 2675
@@
 F 0 "U304" H 6250 4075 50  0000 R CNN
 F 1 "LM833" H 6250 4175 50  0001 R CNN
-F 2 "LM833_Badge:LM833-N-PDIP" H 6025 3875 50  0001 C CNN
+F 2 "SamacSys_Parts:SOIC127P600X175-8N" H 6025 3875 50  0001 C CNN
 F 3 "~" H 6025 3875 50  0001 C CNN
 	3    6025 3875
@@
 F 0 "U301" H 3150 3950 50  0000 R CNN
 F 1 "LM833" H 3175 3975 50  0001 R CNN
-F 2 "LM833_Badge:LM833-N-PDIP" H 2925 3775 50  0001 C CNN
+F 2 "SamacSys_Parts:SOIC127P600X175-8N" H 2925 3775 50  0001 C CNN
 F 3 "~" H 2925 3775 50  0001 C CNN
 	3    2925 3775
@@
 F 0 "U306" H 6125 6025 50  0000 C CNN
 F 1 "LM833" H 6125 6125 50  0000 C CNN
-F 2 "LM833_Badge:LM833-N-PDIP" H 6025 6275 50  0001 C CNN
+F 2 "SamacSys_Parts:SOIC127P600X175-8N" H 6025 6275 50  0001 C CNN
 F 3 "~" H 6025 6275 50  0001 C CNN
 	1    6025 6275
@@
 F 0 "U306" H 6250 6475 50  0000 R CNN
 F 1 "LM833" H 6275 6475 50  0001 R CNN
-F 2 "LM833_Badge:LM833-N-PDIP" H 6025 6275 50  0001 C CNN
+F 2 "SamacSys_Parts:SOIC127P600X175-8N" H 6025 6275 50  0001 C CNN
 F 3 "~" H 6025 6275 50  0001 C CNN
 	3    6025 6275
@@
 F 0 "U307" H 8800 3725 50  0000 C CNN
 F 1 "LM833" H 8800 3825 50  0000 C CNN
-F 2 "LM833_Badge:LM833-N-PDIP" H 8700 3975 50  0001 C CNN
+F 2 "SamacSys_Parts:SOIC127P600X175-8N" H 8700 3975 50  0001 C CNN
 F 3 "~" H 8700 3975 50  0001 C CNN
 	1    8700 3975
@@
 F 0 "U307" H 8950 4150 50  0000 R CNN
 F 1 "LM833" H 8950 4175 50  0001 R CNN
-F 2 "LM833_Badge:LM833-N-PDIP" H 8700 3975 50  0001 C CNN
+F 2 "SamacSys_Parts:SOIC127P600X175-8N" H 8700 3975 50  0001 C CNN
 F 3 "~" H 8700 3975 50  0001 C CNN
 	3    8700 3975
@@
 F 0 "U302" H 6125 1225 50  0000 C CNN
 F 1 "LM833" H 6125 1325 50  0000 C CNN
-F 2 "LM833_Badge:LM833-N-PDIP" H 6025 1475 50  0001 C CNN
+F 2 "SamacSys_Parts:SOIC127P600X175-8N" H 6025 1475 50  0001 C CNN
 F 3 "~" H 6025 1475 50  0001 C CNN
 	1    6025 1475
@@
 F 0 "U302" H 6250 1675 50  0000 R CNN
 F 1 "LM833" H 6275 1675 50  0001 R CNN
-F 2 "LM833_Badge:LM833-N-PDIP" H 6025 1475 50  0001 C CNN
+F 2 "SamacSys_Parts:SOIC127P600X175-8N" H 6025 1475 50  0001 C CNN
 F 3 "~" H 6025 1475 50  0001 C CNN
 	3    6025 1475
@@
 F 0 "U303" H 6250 2875 50  0000 R CNN
 F 1 "LM833" H 6250 2900 50  0001 R CNN
-F 2 "LM833_Badge:LM833-N-PDIP" H 6025 2675 50  0001 C CNN
+F 2 "SamacSys_Parts:SOIC127P600X175-8N" H 6025 2675 50  0001 C CNN
 F 3 "~" H 6025 2675 50  0001 C CNN
 	3    6025 2675
@@
 F 0 "U305" H 6250 5275 50  0000 R CNN
 F 1 "LM833" H 6275 5275 50  0001 R CNN
-F 2 "LM833_Badge:LM833-N-PDIP" H 6025 5075 50  0001 C CNN
+F 2 "SamacSys_Parts:SOIC127P600X175-8N" H 6025 5075 50  0001 C CNN
 F 3 "~" H 6025 5075 50  0001 C CNN
 	3    6025 5075
@@
 F 0 "R327" H 7625 2700 50  0000 C CNN
 F 1 "10k" H 7625 2609 50  0000 C CNN
-F 2 "SamacSys_Parts:RK12L12C0A0G" H 7475 2175 50  0001 C CNN
+F 2 "SamacSys_Parts:3310H001202L" H 7475 2175 50  0001 C CNN
 F 3 "" H 7475 2175 50  0001 C CNN
 	1    7625 2475
@@
 F 0 "R330" H 7625 4100 50  0000 C CNN
 F 1 "1000" H 7625 4009 50  0000 C CNN
-F 2 "SamacSys_Parts:P0925NFC15BR1K" H 7475 3575 50  0001 C CNN
+F 2 "SamacSys_Parts:3310H001202L" H 7475 3575 50  0001 C CNN
 F 3 "" H 7475 3575 50  0001 C CNN
 	1    7625 3875
@@
 F 0 "R332" H 7625 5100 50  0000 C CNN
 F 1 "4000" H 7625 5009 50  0000 C CNN
-F 2 "SamacSys_Parts:RK12L12C0C0P" H 7475 4575 50  0001 C CNN
+F 2 "SamacSys_Parts:3310H001202L" H 7475 4575 50  0001 C CNN
 F 3 "" H 7475 4575 50  0001 C CNN
 	1    7625 4875
@@
 F 0 "R328" H 7625 3225 50  0000 C CNN
 F 1 "1000" H 7625 3150 50  0000 C CNN
-F 2 "SamacSys_Parts:P0925NFC15BR1K" H 7475 2725 50  0001 C CNN
+F 2 "SamacSys_Parts:3310H001202L" H 7475 2725 50  0001 C CNN
 F 3 "" H 7475 2725 50  0001 C CNN
 	1    7625 3025
@@
 F 0 "U304" H 6125 3625 50  0000 C CNN
 F 1 "LM833" H 6125 3725 50  0000 C CNN
-F 2 "LM833_Badge:LM833-N-PDIP" H 6025 3875 50  0001 C CNN
+F 2 "SamacSys_Parts:SOIC127P600X175-8N" H 6025 3875 50  0001 C CNN
 F 3 "~" H 6025 3875 50  0001 C CNN
 	1    6025 3875
