File: FiveStageStereoEQ/FiveStageStereoEQ.sch (KiCad schematic (older format))
At the start: 2 parts, among them J101 AudioJack3, J102 AudioJack3

Commit message: fixed audio jack footprint, added better 3d jack model, added graoe nut logo on bottom silkscree and added gerbers
Parts:
- J101, J102: footprint SamacSys_Parts:SJ13523N -> SJ1-3523N:CUI_SJ1-3523N
Changed lines of the file:
@@
 F 0 "J102" H 8550 3775 50  0000 R CNN
 F 1 "AudioJack3" H 8700 3675 50  0000 R CNN
-F 2 "SamacSys_Parts:SJ13523N" H 8600 4050 50  0001 C CNN
+F 2 "SJ1-3523N:CUI_SJ1-3523N" H 8600 4050 50  0001 C CNN
 F 3 "~" H 8600 4050 50  0001 C CNN
 	1    8600 4050
@@
 F 0 "J101" H 2925 3675 50  0000 C CNN
 F 1 "AudioJack3" H 2925 3575 50  0000 C CNN
-F 2 "SamacSys_Parts:SJ13523N" H 3000 3950 50  0001 C CNN
+F 2 "SJ1-3523N:CUI_SJ1-3523N" H 3000 3950 50  0001 C CNN
 F 3 "~" H 3000 3950 50  0001 C CNN
 	1    3000 3950
